File: Luna65.kicad_sch (KiCad schematic)
At the start: 318 parts, among them J1 TYPE-C-31-M12_13, Q1 DTC123JKAT146, Q2 AO3401A, SW0 SW_Push, SW1 Esc, SW10 9, SW11 0, SW12 -, SW13 =, SW14 BSP_200, SW15 Del, SW16 Tab_150, SW17 Q, SW18 W, SW19 E, SW2 1, SW20 R, SW21 T, SW22 Y, SW23 U, SW24 I, SW25 O, SW26 P, SW27 [, SW28 ], SW29 \_150, SW3 2, SW30 Home, SW31 Caps_175, SW32 A, SW33 S, SW34 D, SW35 F, SW36 G, SW37 H, SW38 J, SW39 K, SW4 3, SW40 L, SW41 ;, SW42 ', SW43 Ent_225, SW44 PgUp, SW45 LShft_225, SW46 Z, SW47 X, SW48 C, SW49 V, SW5 4, SW50 B, SW51 N, SW52 M, SW53 ,, SW54 ., SW55 /, SW56 RShft_175, SW57 Up, SW58 End, SW59 LCtrl_125, SW6 5, SW60 Win_125, SW61 LAlt_125, SW62 Space_625, SW63 RAlt, SW64 Fn, SW65 RCtrl, SW66 Left, SW67 Down, SW68 Right, SW7 6, SW8 7, SW9 8, U1 ATmega32U4-AU, U2 USBLC6-2SC6, Y1 16MHz

Commit message: new changes for v4
Parts:
- removed F1: Polyfuse_Small, Fuse:Fuse_1206_3216Metric_Pad1.42x1.75mm_HandSolder, symbol Device:Polyfuse_Small
- removed H10, H11, H12, H4, H5, H6, H7, H8: MountingHole, MountingHole:MountingHole_2.7mm_M2.5_Pad, symbol Mechanical:MountingHole
- added C14, C15, C16: 10uF, acheron_Components:C_0805_2012Metric, symbol Device:C_Small
- added C17, C18: 1uF, acheron_Components:C_0805_2012Metric, symbol Device:C_Small
- added D139: Green, LED_SMD:LED_1206_3216Metric_Pad1.42x1.75mm_HandSolder, symbol Device:LED_Small
- added D140: Red, LED_SMD:LED_1206_3216Metric_Pad1.42x1.75mm_HandSolder, symbol Device:LED_Small
- added D141: Blue, LED_SMD:LED_1206_3216Metric_Pad1.42x1.75mm_HandSolder, symbol Device:LED_Small
- added J2: JSTPH, Adafruit Feather 32u4 Bluefruit LE:JSTPH2, symbol Connector_Generic:Conn_01x02
- added R80: 10K, Resistor_SMD:R_0805_2012Metric_Pad1.20x1.40mm_HandSolder, symbol Device:R_Small
- added R81: 100K, Resistor_SMD:R_0805_2012Metric_Pad1.20x1.40mm_HandSolder, symbol Device:R_Small
- added R82: 1K, Resistor_SMD:R_0805_2012Metric_Pad1.20x1.40mm_HandSolder, symbol Device:R_Small
- added R83, R84: 2.2K, acheron_Components:R_SMD_1206, symbol Device:R_Small
- added U3: MCP73831, Package_TO_SOT_SMD:SOT-23-5, symbol Battery_Management:MCP73831-2-OT
- added U4: SPX3819M5-L-3-3, Package_TO_SOT_SMD:SOT-23-5, symbol Regulator_Linear:SPX3819M5-L-3-3
- added U5: MBT40, Adafruit Feather 32u4 Bluefruit LE:BLE_MODULE_RAYTAC_MDBT40, symbol Adafruit Feather 32u4 Bluefruit LE-eagle-import:NRF51822_MODULE_MDBT40
- D70: value RB060M-60TR -> MBR120
- R1, R10: value 1k -> 1K
- R11: value 100R -> 100
- R2, R3, R4, R5, R6: footprint acheron_Components:R_SMD_1206 -> Resistor_SMD:R_0805_2012Metric_Pad1.20x1.40mm_HandSolder
- SW62: footprint acheron_MXH:MX625HR -> acheron_MXH:MX625H
- renumbered H9 to H4
Connections:
- net Col10: now also SW29.1 (Col), SW44.1 (Col), U1.26 (PD6); no longer SW63.1 (Col), U1.25 (PD4)
- net Col11: now also U1.27 (PD7); no longer SW64.1 (Col), U1.26 (PD6)
- net Col12: now also U1.29 (PB5); no longer SW65.1 (Col), U1.27 (PD7)
- net Col13: now also U1.30 (PB6); no longer SW13.1 (Col), SW28.1 (Col), SW43.1 (Col), SW66.1 (Col), U1.28 (PB4)
- net Col4: now also U1.12 (PB7); no longer U1.10 (PB2)
- net Col5: now also SW63.1 (Col), SW66.1 (Col), U1.8 (PB0); no longer U1.11 (PB3)
- net Col6: now also SW64.1 (Col), SW67.1 (Col); no longer SW62.1 (Col)
- net Col7: now also SW43.1 (Col), SW65.1 (Col)
- net Col8: now also SW57.1 (Col), SW68.1 (Col)
- net Col9: now also SW28.1 (Col), SW58.1 (Col)
- net GND: now also C14.2, C15.1, C16.2, C17.2, C18.2, D140.1 (K), D141.1 (K), J2.1 (Pin_1), R80.2, U3.2 (VSS), U4.2 (GND), U5.1 (GND@1), U5.13 (GND@3), U5.16 (P0.30), U5.2 (GND@2), U5.25 (GND@4), U5.42 (GND@5); no longer D70.2 (A)
- net Row1: no longer D13.1 (K), D14.1 (K), D15.1 (K)
- net Row2: no longer D28.1 (K), D29.1 (K), D30.1 (K)
- net Row3: no longer D43.1 (K), D44.1 (K)
- net Row4: no longer D57.1 (K), D58.1 (K)
- net Row5: now also D15.1 (K), D30.1 (K), D44.1 (K), D58.1 (K); no longer D66.1 (K), D67.1 (K)
- net VBUS: now also D70.1 (K), C14.1, D139.2 (A), R81.1, U3.4 (VDD), U4.1 (IN)
- net BLE_IRQ: now reaches U1.1 (PE6)
- net BLE_IRQ: now also U5.8 (P0.25)
- net RESET: now reaches C9.1, R9.2, SW0.1, U1.13 (~RESET)
- net SCK: now reaches U1.9 (PB1)
- net SCK: now also U5.4 (P0.21)
- net 5V renamed 3.3V
- net 3.3V: now also C16.1, C17.1, C18.1, U4.5 (OUT), U5.14 (VDD), U5.3 (AVDD); no longer D70.1 (K)
- removed net Col14: SW14.1 (Col), SW29.1 (Col), SW57.1 (Col), SW67.1 (Col), U1.29 (PB5)
- removed net Col15: SW15.1 (Col), SW30.1 (Col), SW44.1 (Col), SW58.1 (Col), SW68.1 (Col), U1.30 (PB6)
- new net: D140.2 (A), R83.2
- new net: R81.2, U4.3 (EN)
- new net: R84.1, U5.39 (P0.19)
- new net: D141.2 (A), R84.2
- new net: R82.1, U3.1 (STAT)
- new net: R80.1, U3.5 (PROG)
- new net: SW14.1 (Col), SW15.1 (Col)
- new net: R83.1, U5.38 (P0.18)
- new net: SW13.1 (Col), SW30.1 (Col)
- new net: D139.1 (K), R82.2
- new net +BATT: C15.2, D70.2 (A), J2.2 (Pin_2), U3.3 (VBAT)
- new net BLE_CS: U1.28 (PB4), U5.7 (P0.24)
- new net MISO: U1.11 (PB3), U5.5 (P0.22)
- new net MOSI: U1.10 (PB2), U5.6 (P0.23)
- new net Row6: D13.1 (K), D14.1 (K), D28.1 (K), D29.1 (K), D43.1 (K), D57.1 (K), D66.1 (K), D67.1 (K)
- new net SWDIO/RST: U1.25 (PD4), U5.35 (SWDIO/NRESET)
- no-connect marks 6 -> 3
Other:
- note added: "1"
- note added: "A"
- note added: "Luna65 Keyboard PCB"
- note added: "USB-C Receptacle"
- note removed: "USB Connector"
- moved on the sheet: C1, C10, C11, C12, C13, C2, C3, C4, C5, C6, C7, C8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

Commit message: Finished V4 routing
Parts:
- added H10, H11, H12, H5, H6, H7, H8, H9: MountingHole, MountingHole:MountingHole_2.7mm_M2.5_Pad, symbol Mechanical:MountingHole
- R1: footprint acheron_Components:R_SMD_1206 -> Resistor_SMD:R_0805_2012Metric_Pad1.20x1.40mm_HandSolder
- SW58: value End -> PgDn
Connections:
- net Col13 is gone; now on net Col11: U1.30 (PB6)
- net Col10: now also SW68.1 (Col), U1.31 (PC6); no longer SW44.1 (Col), U1.26 (PD6)
- net Col11: now also SW13.1 (Col), SW58.1 (Col); no longer U1.27 (PD7)
- net Col12: now also SW30.1 (Col), SW44.1 (Col)
- net Col2: now also U1.19 (PD1); no longer U1.32 (PC7)
- net Col3: now also U1.20 (PD2); no longer U1.31 (PC6)
- net Col4: now also SW62.1 (Col), U1.21 (PD3); no longer U1.12 (PB7)
- net Col5: now also SW28.1 (Col), U1.22 (PD5); no longer SW66.1 (Col), U1.8 (PB0)
- net Col6: now also SW43.1 (Col), U1.26 (PD6); no longer SW67.1 (Col), U1.19 (PD1)
- net Col7: now also SW57.1 (Col), U1.27 (PD7); no longer SW43.1 (Col), U1.20 (PD2)
- net Col8: now also SW15.1 (Col), SW66.1 (Col), U1.12 (PB7); no longer SW57.1 (Col), SW68.1 (Col), U1.21 (PD3)
- net Col9: now also SW14.1 (Col), SW67.1 (Col), U1.32 (PC7); no longer SW28.1 (Col), SW58.1 (Col), U1.22 (PD5)
- net Row1: now also U1.41 (PF0); no longer U1.37 (PF6)
- net Row2: now also U1.40 (PF1); no longer U1.38 (PF5)
- net Row4: now also U1.38 (PF5); no longer U1.40 (PF1)
- net Row5: now also D66.1 (K), D67.1 (K), U1.37 (PF6); no longer D15.1 (K), D30.1 (K), U1.41 (PF0)
- net Row6: now also D15.1 (K), D30.1 (K), U1.8 (PB0); no longer D66.1 (K), D67.1 (K)
Other:
- note added: "9 November 2021"
- note added: "Atmega32u4 Microcontroller"
- note added: "Switch Matrix"
- moved on the sheet: C1, C18, C9, D100, D101, D102, D103, D104, D105, D106, D107, D108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

Commit message: stuff
Parts:
- added G1: MR Logo, Library:MR_logo_sm, symbol Mechanical:MountingHole
- added G2: MR Logo, Library:L6_logo_sm, symbol Mechanical:MountingHole
- Y1: value 16MHz -> 8MHz

Commit message: Rev 5
Parts:
- removed C12, C5, C7: 1uF, acheron_Components:C_0805_2012Metric, symbol Device:C_Small
- removed C6: 10uF, acheron_Components:C_0805_2012Metric, symbol Device:C_Small
- removed C8: 0.1uF, acheron_Components:C_0805_2012Metric, symbol Device:C_Small
- removed D72, D73, D74, D75, D77, D78, D79, D80, D82, D83, D84, D85: LED_Small, LED_SMD:LED_1206_3216Metric_Pad1.42x1.75mm_HandSolder, symbol Device:LED_Small
- removed R1: 1K, Resistor_SMD:R_0805_2012Metric_Pad1.20x1.40mm_HandSolder, symbol Device:R_Small
- removed R12, R13, R14, R15, R18, R19: 420, acheron_Components:R_SMD_1206, symbol Device:R_Small
- removed U1: ATmega32U4-AU, Package_QFP:TQFP-44_10x10mm_P0.8mm, symbol MCU_Microchip_ATmega:ATmega32U4-AU
- added D103, D107, D111, D116, D121, D126, D130, D134, D86, D90, D94, D99: LED_Small, LED_SMD:LED_1206_3216Metric_Pad1.42x1.75mm_HandSolder, symbol Device:LED_Small
- added J3: uC Pin Headers, Connector_PinHeader_1.27mm:PinHeader_2x03_P1.27mm_Vertical, symbol Connector_Generic:Conn_02x03_Odd_Even
- added J4: nRF51 Pin Headers, Connector_PinHeader_1.27mm:PinHeader_2x03_P1.27mm_Vertical, symbol Connector_Generic:Conn_02x03_Odd_Even
- added J5: Pin Headers, Connector_PinHeader_1.27mm:PinHeader_2x01_P1.27mm_Vertical, symbol Connector_Generic:Conn_01x02
- added R22, R27, R80, R81, R82, R83: 100, acheron_Components:R_SMD_1206, symbol Device:R_Small
- added SW69: SW_DPST_x2, symbol Switch:SW_DPST_x2
- added U1: ATMEGA32U4, acheron_Components:TQPF-44_10x10mm_P0.8mm, symbol acheronSymbols:ATMEGA32U4
- C3: value 0.1uF -> 10uF
- C4: value 0.1uF -> 1uF
- G1: footprint Library:MR_logo_sm -> Luna65:MR_logo_sm
- G2: value MR Logo -> Luna Logo; footprint Library:L6_logo_sm -> Luna65:L6_logo_sm
- H4: value MountingHole_Pad -> MountingHole
- R10: renamed from R9; value 10k -> 10K
- R16, R17, R20, R21, R23, R24, R25, R26, R28, R29, R30, R31, R32, R33, R34, R35, R36, R37, R38, R39, R40, R41, R42, R43, R44, R45, R46, R47, R48, R49, R50, R51, R52, R53, R54, R55, R56, R57, R58, R59, R60, R61, R62, R63, R64, R65, R66, R67, R68, R69, R70, R71, R72, R73, R74, R75, R76, R77, R78, R79: value 420 -> 100
- R18: renamed from R22; value 420 -> 100
- R19: renamed from R27; value 420 -> 100
- U4: value SPX3819M5-L-3-3 -> AP2112
- renumbered C15 to C10, C16 to C11, C17 to C12, C18 to C13, C9 to C5, C10 to C6, C11 to C7, C13 to C8, C14 to C9, D76 to D72, D81 to D73, D86 to D74, D90 to D75, D94 to D76, D99 to D77, D103 to D78, D107 to D79, D111 to D80, D116 to D81, D121 to D82, D126 to D83, D130 to D84, D134 to D85, R3 to R1, R8 to R11, R83 to R12, R84 to R13, R10 to R14, R11 to R15, R4 to R2, R2 to R3, R5 to R4, R6 to R5, R80 to R6, R82 to R7, R81 to R8, R7 to R9
Connections:
- net 3.3V: now also J3.2 (Pin_2), U1.14 (VCC), U1.24 (AVCC), U1.33 (~{HWB}/PE2), U1.34 (VCC), U1.44 (AVCC), U1.6 (UCAP); no longer C4.1
- net BLE_CS: now also U1.28 (ADC4/PCINT11/PD8)
- net BLE_IRQ: now also U1.1 (PE6/INT6/AIN0)
- net Col1: now also U1.36 (ADC7/PF7)
- net Col10: now also U1.31 (PC6)
- net Col11: now also U1.30 (PCINT6/ADC13/PB6)
- net Col12: now also U1.29 (PCINT4/ADC12/PB5)
- net Col2: now also U1.19 (PD1/SDA/~{INT1})
- net Col3: now also U1.20 (PD2/RDX1/~{INT2})
- net Col4: now also U1.21 (PD3/TXD1/~{INT3})
- net Col5: now also U1.22 (PD5/~{CTS}/XCK1)
- net Col6: now also U1.26 (ADC9/T1/PD6)
- net Col7: now also U1.27 (ADC10/T0/PD7)
- net Col8: now also U1.12 (PB7/RTS)
- net Col9: now also U1.32 (CLK/PC7)
- net D+: now also U1.4 (D+)
- net D-: now also U1.3 (D-)
- net GND: now also C4.1, D103.1 (K), D107.1 (K), D111.1 (K), D116.1 (K), D121.1 (K), D126.1 (K), D130.1 (K), D134.1 (K), D86.1 (K), D90.1 (K), D94.1 (K), D99.1 (K), J3.6 (Pin_6), J4.6 (Pin_6), U1.15 (GND), U1.23 (GND), U1.35 (GND), U1.43 (GND), U1.5 (UGND); no longer C4.2
- net LED_PWM: now also U1.18 (PD0/SCL/~{INT0})
- net MISO: now also J3.1 (Pin_1), U1.11 (PB3/PDO/PCINT3/MISO)
- net MOSI: now also J3.4 (Pin_4), U1.10 (PB2/PDI/PCINT2/MOSI)
- net RESET: now also J3.5 (Pin_5), U1.13 (~{RESET})
- net Row1: now also U1.41 (ADC0/PF0)
- net Row2: now also U1.40 (ADC1/PF1)
- net Row3: now also U1.39 (ADC4/PF4)
- net Row4: now also U1.38 (ADC5/PF5)
- net Row5: now also U1.37 (ADC5/PF5)
- net Row6: now also U1.8 (PB0/SS/PCINT0)
- net SCK: now also J3.3 (Pin_3), U1.9 (PBI/PCINT1/SCLK)
- net SWDIO/RST: now also J4.3 (Pin_3), U1.25 (ADC8/PD4)
- net VBUS: now also J5.2 (Pin_2), U1.7 (VBUS)
- net at C7.1, Y1.1: now also U1.17 (XTAL1)
- net at C6.1, Y1.2: now also U1.16 (XTAL2)
- net at D84.2 (A): now also R29.2; no longer R71.2
- net at D112.2 (A): now also R57.2; no longer R53.2
- net at D71.2 (A): now also R16.2
- net at Q2.3 (D), R16.1, R17.1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: now also R22.1, R27.1, R80.1, R81.1, R82.1, R83.1
- net at R64.2: now also D119.2 (A); no longer D123.2 (A)
- net at R59.2: now also D114.2 (A); no longer D118.2 (A)
- net at R36.2: now also D91.2 (A); no longer D95.2 (A)
- net at D106.2 (A): now also R51.2; no longer R47.2
- net at D135.2 (A): now also R80.2; no longer R76.2
- net at R65.2: now also D120.2 (A); no longer D124.2 (A)
- net at D88.2 (A): now also R33.2; no longer R29.2
- net at D92.2 (A): now also R37.2; no longer R33.2
- net at D96.2 (A): now also R41.2; no longer R37.2
- net at D104.2 (A): now also R49.2; no longer R45.2
- net at R68.2: now also D123.2 (A); no longer D127.2 (A)
- net at R23.2: now also D78.2 (A)
- net at R32.2: now also D87.2 (A); no longer D91.2 (A)
- net at R60.2: now also D115.2 (A); no longer D119.2 (A)
- net at R42.2: now also D97.2 (A); no longer D101.2 (A)
- net at D79.2 (A): now also R24.2; no longer R48.2
- net at D81.2 (A): now also R26.2; no longer R57.2
- net at D108.2 (A): now also R53.2; no longer R49.2
- net at D80.2 (A): now also R25.2; no longer R52.2
- net at R28.2: now also D83.2 (A); no longer D87.2 (A)
- net at R61.2: now also D116.2 (A); no longer D120.2 (A)
- net at D131.2 (A): now also R76.2; no longer R72.2
- net at D136.2 (A): now also R81.2; no longer R77.2
- net at D113.2 (A): now also R58.2; no longer R54.2
- net at R20.2: now also D75.2 (A)
- net at D133.2 (A): now also R78.2; no longer R74.2
- net at R73.2: now also D128.2 (A); no longer D132.2 (A)
- net at R55.2: now also D110.2 (A); no longer D114.2 (A)
- net at D117.2 (A): now also R62.2; no longer R58.2
- net at D82.2 (A): now also R27.2; no longer R62.2
- net DFU: now reaches U5.24 (P0.07)
- net DFU: now also J4.4 (Pin_4)
- net FCTRYRST: now reaches U5.34 (P0.16)
- net FCTRYRST: now also J4.5 (Pin_5)
- net SWCLK: now reaches U5.36 (SWCLK)
- net SWCLK: now also J4.1 (Pin_1)
- net at R30.2: now also D85.2 (A); no longer D89.2 (A)
- net at R21.2: now also D76.2 (A)
- net at R50.2: now also D105.2 (A); no longer D109.2 (A)
- net at R75.2: now also D130.2 (A); no longer D85.2 (A)
- net at R46.2: now also D101.2 (A); no longer D105.2 (A)
- net at R44.2: now also D99.2 (A); no longer D78.2 (A)
- net at R70.2: now also D125.2 (A); no longer D129.2 (A)
- net at R66.2: now also D121.2 (A); no longer D125.2 (A)
- net at D122.2 (A): now also R67.2; no longer R63.2
- net at R79.2: now also D134.2 (A); no longer D138.2 (A)
- net at R35.2: now also D90.2 (A); no longer D76.2 (A)
- net at R56.2: now also D111.2 (A); no longer D115.2 (A)
- net at D93.2 (A): now also R38.2; no longer R34.2
- net at D137.2 (A): now also R82.2; no longer R78.2
- net at R43.2: now also D98.2 (A); no longer D102.2 (A)
- net at R40.2: now also D95.2 (A); no longer D77.2 (A)
- net at D100.2 (A): now also R45.2; no longer R41.2
- net at R31.2: now also D86.2 (A); no longer D75.2 (A)
- net at R39.2: now also D94.2 (A); no longer D98.2 (A)
- net at R69.2: now also D124.2 (A); no longer D128.2 (A)
- net +BATT renamed VBAT
- net VBAT: now also J5.1 (Pin_1)
- new net: C4.2, U1.42 (AREF)
- new net: D107.2 (A), R52.2
- new net: D126.2 (A), R71.2
- new net: D138.2 (A), R83.2
- new net: D103.2 (A), R48.2
- new net: D109.2 (A), R54.2
- new net: D129.2 (A), R74.2
- new net: D132.2 (A), R77.2
- new net: D89.2 (A), R34.2
- new net: D127.2 (A), R72.2
- new net: D77.2 (A), R22.2
- new net: D118.2 (A), R63.2
- new net: D102.2 (A), R47.2
- no-connect marks 3 -> 4
Other:
- note added: "25 November 2021"
- note added: "3.3V LDO Regulator"
- note added: "Bluetooth Module"
- note added: "CASE to GND"
- note added: "Graphics"
- note added: "LED Matrix"
- note added: "LiPo Charge Controller"
- note added: "Microcontroller"
- note added: "Mounting Holes"
- note added: "Reset Switch Circuit"
- note added: "USB ESD Protection"
- note removed: "9 November 2021"
- note removed: "Atmega32u4 Microcontroller"
- moved on the sheet: C1, C10, C11, C12, C13, C2, C5, C6, C7, C8, C9, D1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
