File: Luna65.kicad_sch (KiCad schematic)
At the start: 334 parts, among them J1 TYPE-C-31-M12_13, J2 JSTPH, J3 uC Pin Headers, J4 nRF51 Pin Headers, J5 Pin Headers, Q1 DTC123JKAT146, Q2 AO3401A, SW0 SW_Push, SW1 Esc, SW10 9, SW11 0, SW12 -, SW13 =, SW14 BSP_200, SW15 Del, SW16 Tab_150, SW17 Q, SW18 W, SW19 E, SW2 1, SW20 R, SW21 T, SW22 Y, SW23 U, SW24 I, SW25 O, SW26 P, SW27 [, SW28 ], SW29 \_150, SW3 2, SW30 Home, SW31 Caps_175, SW32 A, SW33 S, SW34 D, SW35 F, SW36 G, SW37 H, SW38 J, SW39 K, SW4 3, SW40 L, SW41 ;, SW42 ', SW43 Ent_225, SW44 PgUp, SW45 LShft_225, SW46 Z, SW47 X, SW48 C, SW49 V, SW5 4, SW50 B, SW51 N, SW52 M, SW53 ,, SW54 ., SW55 /, SW56 RShft_175, SW57 Up, SW58 PgDn, SW59 LCtrl_125, SW6 5, SW60 Win_125, SW61 LAlt_125, SW62 Space_625, SW63 RAlt, SW64 Fn, SW65 RCtrl, SW66 Left, SW67 Down, SW68 Right, SW69 SW_DPST_x2, SW7 6, SW8 7, SW9 8, U1 ATMEGA32U4, U2 USBLC6-2SC6, U3 MCP73831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

Commit message: Fixed Broken Bluetooth
Parts:
- removed C11: 10uF, acheron_Components:C_0805_2012Metric, symbol Device:C_Small
- removed SW69: SW_DPST_x2, symbol Switch:SW_DPST_x2
Connections:
- net BLE_CS: now also U1.8 (PB0/SS/PCINT0); no longer U1.28 (ADC4/PCINT11/PD8)
- net Row6: now also U1.28 (ADC4/PCINT11/PB4); no longer U1.8 (PB0/SS/PCINT0)

Commit message: Update Schematic Ver
Other:
- note added: "5"
- note added: "7 December 2021"
- note removed: "25 November 2021"
- note removed: "A"
Changed lines of the file:
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@@
     (effects (font (size 1.778 1.778)) (justify left bottom))
   )
-  (text "A" (at 448.945 284.099 0)
+  (text "5" (at 448.945 284.099 0)
     (effects (font (size 1.27 1.27)) (justify left bottom))
   )
@@
     (effects (font (size 1.778 1.778)) (justify left bottom))
   )
-  (text "25 November 2021" (at 386.588 283.972 0)
+  (text "7 December 2021" (at 386.588 283.972 0)
     (effects (font (size 1.27 1.27)) (justify left bottom))
   )
