File: kicad_files/Luna65-Daughter-Board.kicad_sch (KiCad schematic)
At the start: 29 parts, among them J1 TYPE-C-31-M12_13, J2 Molex Power, J3 JSTPH, J4 Pin Header, U1 MCP73831, U2 USBLC6-2SC6, U3 AP2112

Commit message: DB Rev B
Parts:
- removed H2, H3: MountingHole, MountingHole:MountingHole_2.2mm_M2, symbol Mechanical:MountingHole
- removed J4: Pin Header, Connector_PinHeader_1.27mm:PinHeader_1x03_P1.27mm_Vertical, symbol Connector_Generic:Conn_01x03
- added C10: 22uF, acheron_Components:C_0805_2012Metric, symbol Device:C_Small
- added C8: 10uF, acheron_Components:C_0805_2012Metric, symbol Device:C_Small
- added C9: 1uF, acheron_Components:C_0805_2012Metric, symbol Device:C_Small
- added D4: MBR120, acheron_Components:D_SOD-123, symbol Device:D_Schottky_Small
- added L1: LPS3015-222ML, Luna65:LPS3015, symbol Device:L
- added R10: 3.6M, Resistor_SMD:R_0805_2012Metric, symbol Device:R_Small
- added R11: 261K, Resistor_SMD:R_0805_2012Metric, symbol Device:R_Small
- added U4: TPS61202DRC, Package_SON:Texas_S-PVSON-N10_ThermalVias, symbol Regulator_Switching:TPS61202DRC
- R1, R2, R3, R4, R5, R6, R7, R8, R9: footprint Resistor_SMD:R_0805_2012Metric_Pad1.20x1.40mm_HandSolder -> Resistor_SMD:R_0805_2012Metric
- renumbered H4 to H2
Connections:
- net 3.3V: now also J2.3 (Pin_3); no longer J2.1 (Pin_1)
- net D+: now also J2.2 (Pin_2); no longer J2.4 (Pin_4)
- net D-: now also J2.1 (Pin_1); no longer J2.3 (Pin_3)
- net GND: now also C10.2, C8.2, C9.2, R11.2, U4.11 (PAD), U4.4 (PGND), U4.9 (GND)
- net VBAT: now also C8.1, L1.1, R10.1, U4.5 (VIN), U4.6 (EN), U4.8 (PS); no longer D2.2 (A)
- net VBUS renamed VUSB
- net VUSB: now also D4.2 (A); no longer C4.1, D2.1 (K), J2.2 (Pin_2), R8.1, U3.1 (IN)
- new net: R10.2, R11.1, U4.7 (UVLO)
- new net: C10.1, D2.2 (A), U4.10 (FB), U4.2 (VOUT)
- new net: C9.1, U4.1 (VAUX)
- new net: L1.2, U4.3 (L)
- new net 5V: C4.1, D2.1 (K), D4.1 (K), J2.4 (Pin_4), R8.1, U3.1 (IN)
Other:
- note added: "5V Boost IC"
- note removed: "Mounting Holes"
- company: (none) -> Neil Khera
- title: (none) -> Luna65 Daughter Board
- moved on the sheet: C1, C2, C4, C5, C6, D1, D2, D3, H1, H2, J1, J2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

Commit message: DB Rev C
Parts:
- removed D2, D4: MBR120, acheron_Components:D_SOD-123, symbol Device:D_Schottky_Small
- removed U4: TPS61202DRC, Package_SON:Texas_S-PVSON-N10_ThermalVias, symbol Regulator_Switching:TPS61202DRC
- added C7: 0.1uF, acheron_Components:C_0805_2012Metric, symbol Device:C_Small
- added D2: Red, LED_SMD:LED_1206_3216Metric_Pad1.42x1.75mm_HandSolder, symbol Device:LED_Small
- added Q1: MMUN2133LT1G, Package_TO_SOT_SMD:SOT-23, symbol Transistor_BJT:MMBTA92
- added R12: 100K, Resistor_SMD:R_0805_2012Metric, symbol Device:R_Small
- added R13: 1K, Resistor_SMD:R_0805_2012Metric, symbol Device:R_Small
- added U4: APX803L, Package_TO_SOT_SMD:SOT-23, symbol Power_Management:BD49KxxG
- added U5: TPS61032RSAR, Package_DFN_QFN:Texas_S-PVQFN-N16_EP2.7x2.7mm_ThermalVias, symbol TPS61030PWP:TPS61030PWP
- C10: value 22uF -> 220uF; footprint acheron_Components:C_0805_2012Metric -> Capacitor_SMD:C_1206_3216Metric
- C9: value 1uF -> 2.2uF
- J1: value TYPE-C-31-M12_13 -> TYPE-C-31-M12; symbol acheronSymbols:TYPE-C-31-M12_13 -> acheron_Symbols:TYPE-C-31-M-12
- L1: value LPS3015-222ML -> 6.8uH XAL4030; footprint Luna65:LPS3015 -> Luna65:XAL4030
- R10: value 3.6M -> 2.34M
- R11: value 261K -> 390K
- R4: value 10K -> 1K
Connections:
- net 3.3V: now also J2.1 (Pin_1); no longer J2.3 (Pin_3)
- net 5V: now also C10.1, C9.1, J2.2 (Pin_2), U5.13 (VOUT), U5.14 (VOUT), U5.15 (VOUT); no longer J2.4 (Pin_4)
- net D+: now also J2.4 (Pin_4); no longer J2.2 (Pin_2)
- net D-: now also J2.3 (Pin_3); no longer J2.1 (Pin_1)
- net GND: now also C7.2, D2.1 (K), U4.1 (GND), U5.11 (GND), U5.17 (PGND), U5.18 (PGND), U5.19 (PGND), U5.20 (PGND), U5.21 (PGND), U5.22 (PGND), U5.23 (PGND), U5.24 (PGND), U5.25 (PGND), U5.26 (PGND), U5.27 (PGND), U5.28 (PGND), U5.29 (PGND), U5.3 (PGND), U5.4 (PGND), U5.5 (PGND), U5.8 (SYNC)
- net SHIELD: now also J1.S1 (SHIELD); no longer J1.S (SHIELD)
- net VBAT: now also C7.1, Q1.2 (E), R12.1, U4.3 (VDD), U5.6 (VBAT)
- net at R10.2, R11.1: now also U5.7 (LBI)
- net at L1.2: now also U5.1 (SW), U5.2 (SW)
- new net: Q1.3 (C), R13.1
- new net: D2.2 (A), R13.2
- new net EN: R12.2, U4.2 (VOUT), U5.9 (EN)
- new net LBO: Q1.1 (B), U5.10 (LBO)
- no-connect marks 3 -> 4
Other:
- moved on the sheet: C1, C2, C3, C4, C5, C6, D1, D3, H1, H2, J2, J3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

Commit message: Added 0 Ohm resistor to isolate BT and uC 3.3V
Parts:
- R2: value 5.1k -> 5.1K
Changed lines of the file:
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@@
     (in_bom yes) (on_board yes)
     (property "Reference" "R2" (id 0) (at 52.324 28.702 90))
-    (property "Value" "5.1k" (id 1) (at 52.324 30.734 90)
+    (property "Value" "5.1K" (id 1) (at 52.324 30.734 90)
       (effects (font (size 0.7874 0.7874)))
     )
@@
     )
     (path "/af35a153-e4cc-4cb5-9b0a-a247aa9a27b2"
-      (reference "R2") (unit 1) (value "5.1k") (footprint "Resistor_SMD:R_0805_2012Metric")
+      (reference "R2") (unit 1) (value "5.1K") (footprint "Resistor_SMD:R_0805_2012Metric")
     )
     (path "/56dc9d1a-d125-4218-be7e-afbadad9f13c"

Commit message: Limit RGB max brightness
Parts:
- R4: value 1K -> 2K
- U5: footprint Package_DFN_QFN:Texas_S-PVQFN-N16_EP2.7x2.7mm_ThermalVias -> Package_DFN_QFN:Texas_S-PVQFN-N16_EP2.7x2.7mm; symbol TPS61030PWP:TPS61030PWP -> TPS61032RSAR:TPS61032RSAR
Connections:
- net 5V: now also U5.1 (VOUT), U5.16 (VOUT); no longer U5.13 (VOUT), U5.14 (VOUT)
- net EN: now also U5.11 (EN); no longer U5.9 (EN)
- net GND: now also U5.10 (SYNC), U5.13 (GND), U5.6 (PGND), U5.7 (PGND); no longer U5.11 (GND), U5.18 (PGND), U5.19 (PGND), U5.20 (PGND), U5.21 (PGND), U5.22 (PGND), U5.23 (PGND), U5.24 (PGND), U5.25 (PGND), U5.26 (PGND), U5.27 (PGND), U5.28 (PGND), U5.29 (PGND), U5.3 (PGND), U5.4 (PGND), U5.8 (SYNC)
- net LBO: now also U5.12 (LBO); no longer U5.10 (LBO)
- net VBAT: now also U5.8 (VBAT); no longer U5.6 (VBAT)
- net at R10.2, R11.1: now also U5.9 (LBI); no longer U5.7 (LBI)
- new net: L1.2, U5.3 (SW), U5.4 (SW)
Changed lines of the file:
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@@
       (effects (font (size 1.27 1.27)) (justify left))
     )
-    (property "Value" "1K" (id 1) (at 71.755 48.514 90)
+    (property "Value" "2K" (id 1) (at 71.755 48.514 90)
       (effects (font (size 0.762 0.762)) (justify left))
     )
@@
     (pin "1")
   )
-  (symbol (lib_id "TPS61030PWP:TPS61030PWP") (at 92.202 90.424 0) (unit 1)
+  (symbol (lib_id "TPS61032RSAR:TPS61032RSAR") (at 92.202 90.424 0) (unit 1)
     (in_bom yes) (on_board yes) (fields_autoplaced)
     (property "Reference" "U5" (id 0) (at 87.757 71.4842 0))
     (property "Value" "TPS61032RSAR" (id 1) (at 87.757 74.0211 0))
-    (property "Footprint" "Package_DFN_QFN:Texas_S-PVQFN-N16_EP2.7x2.7mm_ThermalVias" (id 2) (at 76.962 100.584 0)
+    (property "Footprint" "Package_DFN_QFN:Texas_S-PVQFN-N16_EP2.7x2.7mm" (id 2) (at 76.962 100.584 0)
       (effects (font (size 1.27 1.27)) (justify left bottom) hide)
     )
@@
     (pin "14")
     (pin "15")
+    (pin "16")
     (pin "17")
-    (pin "18")
-    (pin "19")
-    (pin "2")
-    (pin "20")
-    (pin "21")
-    (pin "22")
-    (pin "23")
-    (pin "24")
-    (pin "25")
-    (pin "26")
-    (pin "27")
-    (pin "28")
-    (pin "29")
     (pin "3")
     (pin "4")
@@
     )
     (path "/60472c1b-d631-4f5d-b928-0950c0b0a31e"
-      (reference "R4") (unit 1) (value "1K") (footprint "Resistor_SMD:R_0805_2012Metric")
+      (reference "R4") (unit 1) (value "2K") (footprint "Resistor_SMD:R_0805_2012Metric")
     )
     (path "/b2ca14c3-9645-4c6b-8d7c-fa1223882a76"
@@
     )
     (path "/7803dbd1-1d02-40a8-89a2-dd5788ff191f"
-      (reference "U5") (unit 1) (value "TPS61032RSAR") (footprint "Package_DFN_QFN:Texas_S-PVQFN-N16_EP2.7x2.7mm_ThermalVias")
-    )
-  )
+      (reference "U5") (unit 1) (value "TPS61032RSAR") (footprint "Package_DFN_QFN:Texas_S-PVQFN-N16_EP2.7x2.7mm")
+    )
+  )

Commit message: DB Rev 4 Changes
Parts:
- removed Q1: MMUN2133LT1G, Package_TO_SOT_SMD:SOT-23, symbol Transistor_BJT:MMBTA92
- removed U1: MCP73831, Package_TO_SOT_SMD:SOT-23-5, symbol Battery_Management:MCP73831-2-OT
- added Q1: TP0610T, Package_TO_SOT_SMD:SOT-23, symbol Transistor_FET:TP0610T
- added R14: 1K, Resistor_SMD:R_0805_2012Metric, symbol Device:R_Small
- added U6: LTC4095, Package_DFN_QFN:DFN-8-1EP_2x2mm_P0.5mm_EP0.7x1.3mm, symbol LTC4095:LTC4095
- C2: value 10uF -> 1uF
- R4: value 2K -> 1K
- R6: value 1K -> 842
Connections:
- net 5V: now also Q1.2 (S), R14.1
- net GND: now also C2.2, R6.2, U6.2 (GND), U6.4 (SUSP), U6.6 (NTC), U6.9 (GND); no longer C2.1, R4.2
- net LBO: now also Q1.1 (G), R14.2
- net VBAT: now also U6.1 (BAT); no longer C2.2
- net VUSB: now also C2.1, U6.5 (HPWR), U6.8 (IN)
- net at R13.1: now also Q1.3 (D)
- net at R6.1: now also U6.7 (PROG)
- net at D1.1 (K): now also R4.2; no longer R6.2
- net at R4.1: now also U6.3 (CHRG)
Other:
- moved on the sheet: C10, C7, C9, D2, J3, R12, R13, U4

Commit message: stuff
Parts:
- removed U6: LTC4095, Package_DFN_QFN:DFN-8-1EP_2x2mm_P0.5mm_EP0.7x1.3mm, symbol LTC4095:LTC4095
- added C11, C12: 10uF, Capacitor_SMD:C_0603_1608Metric, symbol Device:C_Small
- added L2: 1.5uH, Inductor_SMD:L_0805_2012Metric, symbol Device:L_Small
- added U1: LTC4001, Package_DFN_QFN:QFN-16-1EP_4x4mm_P0.65mm_EP2.15x2.15mm, symbol Battery_Management:LTC4001
- C1, C3, C4, C5, C6, C7, C8, C9: footprint acheron_Components:C_0805_2012Metric -> Capacitor_SMD:C_0603_1608Metric
- C2: value 1uF -> 0.1uF; footprint acheron_Components:C_0805_2012Metric -> Capacitor_SMD:C_0603_1608Metric
- D1, D2: footprint LED_SMD:LED_1206_3216Metric_Pad1.42x1.75mm_HandSolder -> LED_SMD:LED_0805_2012Metric
- R1, R10, R11, R12, R13, R14, R2, R3, R4, R5, R7, R8, R9: footprint Resistor_SMD:R_0805_2012Metric -> Resistor_SMD:R_0603_1608Metric
- R6: value 842 -> 274; footprint Resistor_SMD:R_0805_2012Metric -> Resistor_SMD:R_0603_1608Metric
Connections:
- net GND: now also R6.1, C11.2, C12.2, U1.11 (NTC), U1.15 (TIMER), U1.17 (PAD), U1.3 (PGND), U1.4 (GNDSENS), U1.6 (~{EN}); no longer R6.2
- net VBAT: now also C12.1, U1.1 (BAT), U1.16 (BATSENS)
- net VUSB: now also C11.1, U1.8 (PVin), U1.9 (Vinsense); no longer C2.1
- net at R4.1: now also U1.7 (~{CHRG})
- new net: L2.1, U1.5 (SW)
- new net: L2.2, U1.2 (SENSE)
- new net: R6.2, U1.12 (PROG), U1.13 (IDET)
- new net: C2.1, U1.14 (SS)
- no-connect marks 4 -> 5
Other:
- moved on the sheet: D1, R4

Commit message: DB Rev 8
Parts:
- removed L2: 1.5uH, Inductor_SMD:L_0805_2012Metric, symbol Device:L_Small
- removed U1: LTC4001, Package_DFN_QFN:QFN-16-1EP_4x4mm_P0.65mm_EP2.15x2.15mm, symbol Battery_Management:LTC4001
- added R15: 10K, Resistor_SMD:R_0603_1608Metric, symbol Device:R_Small
- added R16: 1K, Resistor_SMD:R_0603_1608Metric, symbol Device:R_Small
- added R17: 1.5K, Resistor_SMD:R_0603_1608Metric, symbol Device:R_Small
- added U1: BQ24074RGT, Package_DFN_QFN:VQFN-16-1EP_3x3mm_P0.5mm_EP1.6x1.6mm, symbol Battery_Management:BQ24074RGT
- C11, C12: value 10uF -> 4.7uF
- C2: value 0.1uF -> 1uF
- D1: value Green -> Orange
- R10: value 2.34M -> 2.43M
- R4: value 1K -> 8K
- R6: value 274 -> 10K
- U4: value APX803L -> APX803L-35
Connections:
- net 5V: no longer C4.1, R8.1, U3.1 (IN)
- net GND: now also C11.1, C12.1, C2.1, R4.1, R15.2, R17.1, U1.14 (TMR), U1.17 (VSS), U1.4 (~{CE}), U1.6 (EN1), U1.8 (VSS); no longer C11.2, C12.2, C2.2
- net at R6.2: now also U1.15 (ITERM)
- net at R4.2: now also U1.16 (ISET); no longer D1.1 (K)
- net VBAT renamed VCC
- net VCC: now also C12.2, C4.1, R8.1, U3.1 (IN), R16.2, U1.10 (OUT), U1.11 (OUT), U1.5 (EN2); no longer C12.1, J3.2 (Pin_2)
- net VUSB renamed VBUS
- net VBUS: now also C2.2, U1.13 (IN); no longer C11.1, D1.2 (A)
- new net: R15.1, U1.1 (TS)
- new net: R17.2, U1.12 (ILIM)
- new net: D1.1 (K), U1.9 (~{CHG})
- new net: D1.2 (A), R16.1
- new net +BATT: C11.2, J3.2 (Pin_2), U1.2 (BAT), U1.3 (BAT)
Other:
- moved on the sheet: C3, J3
